Commit message: Fix missing joint axis consideration in joint transform
In particular the transform from the frame indicating the joint position in the parent link to the frame of the child link is dependent on the joint axis

File: URDFs/iCub_r_leg.urdf (robot description, URDF)
Before this commit: robot iDynTreeURDFModelExportModelName, 7 links, 6 joints
Links:
- added link base_link
- added link chest
- added link head
- added link l_ankle_1
- added link l_ankle_2
- added link l_arm_ft_sensor
- added link l_elbow_1
- added link l_foot_front
- added link l_foot_front_ft_sensor
- added link l_foot_rear
- added link l_foot_rear_ft_sensor
- added link l_forearm
- added link l_hand
- added link l_hip_1
- added link l_hip_2
- added link l_hip_3
- added link l_leg_ft_sensor
- added link l_lower_leg
- added link l_shoulder_1
- added link l_shoulder_2
- added link l_shoulder_3
- added link l_sole
- added link l_upper_arm
- added link l_upper_leg
- added link l_wrist_1
- added link neck_1
- added link neck_2
- added link neck_3
- added link r_arm_ft_sensor
- added link r_elbow_1
- added link r_foot_front
- added link r_foot_front_ft_sensor
- added link r_foot_rear
- added link r_foot_rear_ft_sensor
- added link r_forearm
- added link r_hand
- added link r_hip_3
- added link r_leg_ft_sensor
- added link r_shoulder_1
- added link r_shoulder_2
- added link r_shoulder_3
- added link r_sole
- added link r_upper_arm
- added link r_wrist_1
- added link torso_1
- added link torso_2
Joints:
- added joint base_link_fixed_joint: type fixed, parent root_link, child base_link, origin xyz=0 0 0 rpy=0 -0 0
- added joint chest_fixed_joint: type fixed, parent root_link, child chest, origin xyz=0 0 0.19747000000000003 rpy=0 -0 0
- added joint head_fixed_joint: type fixed, parent root_link, child head, origin xyz=0.0048615099999999994 0 0.4904200000000001 rpy=0 -0 0
- added joint l_ankle_1_fixed_joint: type fixed, parent root_link, child l_ankle_1, origin xyz=0.026049999999999997 0.08295000000000001 -0.5317890000000001 rpy=0 -0 0
- added joint l_ankle_2_fixed_joint: type fixed, parent root_link, child l_ankle_2, origin xyz=-0.02670000000000001 0.06475 -0.5667890000000001 rpy=0 -0 0
- added joint l_arm_ft_sensor_fixed_joint: type fixed, parent root_link, child l_arm_ft_sensor, origin xyz=0.01160250023188351 0.14719399989874468 0.2765873999902195 rpy=0.0790794230156212 -0.052031613930206826 -0.27527862099575323
- added joint l_elbow_1_fixed_joint: type fixed, parent root_link, child l_elbow_1, origin xyz=0.031246122657570638 0.15209302229214877 0.13144299586628905 rpy=0.0790794230156212 -0.052031613930206826 -0.27527862099575323
- added joint l_foot_front_fixed_joint: type fixed, parent root_link, child l_foot_front, origin xyz=0.10854999999999998 0.06475 -0.6325890000000001 rpy=0 -0 0
- added joint l_foot_front_ft_sensor_fixed_joint: type fixed, parent root_link, child l_foot_front_ft_sensor, origin xyz=0.10854999999999998 0.06475 -0.6325890000000001 rpy=0 -0 0
- added joint l_foot_rear_fixed_joint: type fixed, parent root_link, child l_foot_rear, origin xyz=-0.010700000000000008 0.06475 -0.6325890000000001 rpy=0 -0 0
- added joint l_foot_rear_ft_sensor_fixed_joint: type fixed, parent root_link, child l_foot_rear_ft_sensor, origin xyz=-0.010700000000000008 0.06475 -0.6325890000000001 rpy=0 -0 0
- added joint l_forearm_fixed_joint: type fixed, parent root_link, child l_forearm, origin xyz=0.021311022773212826 0.16151002194112832 0.07576799578628049 rpy=0.0790794230156212 -0.052031613930206826 -0.27527862099575323
- added joint l_hand_fixed_joint: type fixed, parent root_link, child l_hand, origin xyz=0.027938017812163745 0.16329101706262705 -0.031628925986897 rpy=0.0790794230156212 -0.052031613930206826 -0.27527862099575323
- added joint l_hip_1_fixed_joint: type fixed, parent root_link, child l_hip_1, origin xyz=0.0216 0.04045000000000001 0 rpy=0 -0 0
- added joint l_hip_2_fixed_joint: type fixed, parent root_link, child l_hip_2, origin xyz=-0.02565 0.07355 -0.009000000000000008 rpy=0 -0 0
- added joint l_hip_3_fixed_joint: type fixed, parent root_link, child l_hip_3, origin xyz=0.011049999999999997 0.07355 -0.09869999999999995 rpy=0 -0 0
- added joint l_leg_ft_sensor_fixed_joint: type fixed, parent root_link, child l_leg_ft_sensor, origin xyz=0.011049999999999997 0.07355 -0.09869999999999995 rpy=0 -0 0
- added joint l_lower_leg_fixed_joint: type fixed, parent root_link, child l_lower_leg, origin xyz=0.026049999999999997 0.08345000000000001 -0.2758 rpy=0 -0 0
- added joint l_shoulder_1_fixed_joint: type fixed, parent root_link, child l_shoulder_1, origin xyz=-0.020835100000000002 0.0397423 0.3026729 rpy=0.2532616237670649 -1.1982921379466467e-7 -0.26179930185680106
- added joint l_shoulder_2_fixed_joint: type fixed, parent root_link, child l_shoulder_2, origin xyz=0.011907900000000013 0.14265000000000003 0.3308707 rpy=0.0790794230156212 -0.052031613930206826 -0.27527862099575323
- added joint l_shoulder_3_fixed_joint: type fixed, parent root_link, child l_shoulder_3, origin xyz=0.01160250023188351 0.14719399989874468 0.2765873999902195 rpy=0.0790794230156212 -0.052031613930206826 -0.27527862099575323
- added joint l_sole_fixed_joint: type fixed, parent root_link, child l_sole, origin xyz=0.048929999999999994 0.06475 -0.6325890000000001 rpy=0 -0 0
- added joint l_upper_arm_fixed_joint: type fixed, parent root_link, child l_upper_arm, origin xyz=0.013208121959356507 0.14858702204000246 0.2541880957564809 rpy=0.0790794230156212 -0.052031613930206826 -0.27527862099575323
- added joint l_upper_leg_fixed_joint: type fixed, parent root_link, child l_upper_leg, origin xyz=0.011049999999999997 0.05855 -0.16960000000000003 rpy=0 -0 0
- added joint l_wrist_1_fixed_joint: type fixed, parent root_link, child l_wrist_1, origin xyz=0.04547212334915017 0.1655890223793864 -0.030229004065574397 rpy=0.0790794230156212 -0.052031613930206826 -0.27527862099575323
- added joint neck_1_fixed_joint: type fixed, parent root_link, child neck_1, origin xyz=-0.00378849 0 0.3627695 rpy=0 -0 0
- added joint neck_2_fixed_joint: type fixed, parent root_link, child neck_2, origin xyz=0.0048615099999999994 0 0.4117695 rpy=0 -0 0
- added joint neck_3_fixed_joint: type fixed, parent root_link, child neck_3, origin xyz=0.0048615099999999994 0 0.42127000000000003 rpy=0 -0 0
- added joint r_arm_ft_sensor_fixed_joint: type fixed, parent root_link, child r_arm_ft_sensor, origin xyz=0.011602500000000036 -0.14719400000000007 0.27658740000000004 rpy=-0.07907934249382903 -0.0520316044795478 0.2752784843541201
- added joint r_elbow_1_fixed_joint: type fixed, parent root_link, child r_elbow_1, origin xyz=0.031246121282148414 -0.1520930222338017 0.13144299574009638 rpy=-0.07907934249382903 -0.0520316044795478 0.2752784843541201
- added joint r_foot_front_fixed_joint: type fixed, parent r_ankle_2, child r_foot_front, origin xyz=0.13525 0 -0.06579999999999997 rpy=0 -0 0
- added joint r_foot_front_ft_sensor_fixed_joint: type fixed, parent r_ankle_2, child r_foot_front_ft_sensor, origin xyz=0.13525 0 -0.06579999999999997 rpy=0 -0 0
- added joint r_foot_rear_fixed_joint: type fixed, parent r_ankle_2, child r_foot_rear, origin xyz=0.016 0 -0.06579999999999997 rpy=0 -0 0
- added joint r_foot_rear_ft_sensor_fixed_joint: type fixed, parent r_ankle_2, child r_foot_rear_ft_sensor, origin xyz=0.016 0 -0.06579999999999997 rpy=0 -0 0
- added joint r_forearm_fixed_joint: type fixed, parent root_link, child r_forearm, origin xyz=0.021311021282148408 -0.16151002223380165 0.0757679957400964 rpy=-0.07907934249382903 -0.0520316044795478 0.2752784843541201
- added joint r_hand_fixed_joint: type fixed, parent root_link, child r_hand, origin xyz=0.027649815623035374 -0.16337301732292386 -0.031644925317804405 rpy=-0.07907934249382903 -0.0520316044795478 0.2752784843541201
- added joint r_hip_3_fixed_joint: type fixed, parent r_hip_2, child r_hip_3, origin xyz=0.036699999999999997 0 -0.08969999999999995 rpy=0 -0 0
- added joint r_leg_ft_sensor_fixed_joint: type fixed, parent r_hip_2, child r_leg_ft_sensor, origin xyz=0.036699999999999997 0 -0.08969999999999995 rpy=0 -0 0
- added joint r_shoulder_1_fixed_joint: type fixed, parent root_link, child r_shoulder_1, origin xyz=-0.020835100000000002 -0.0397423 0.3026729 rpy=-0.25326164431680925 2.3014774394592079e-7 0.26179970938509745
- added joint r_shoulder_2_fixed_joint: type fixed, parent root_link, child r_shoulder_2, origin xyz=0.014310500000000032 -0.14197200000000007 0.33100070000000004 rpy=-0.07907934249382903 -0.0520316044795478 0.2752784843541201
- added joint r_shoulder_3_fixed_joint: type fixed, parent root_link, child r_shoulder_3, origin xyz=0.011602500000000036 -0.14719400000000007 0.27658740000000004 rpy=-0.07907934249382903 -0.0520316044795478 0.2752784843541201
- added joint r_sole_fixed_joint: type fixed, parent r_ankle_2, child r_sole, origin xyz=0.07563 0 -0.06579999999999997 rpy=0 -0 0
- added joint r_upper_arm_fixed_joint: type fixed, parent root_link, child r_upper_arm, origin xyz=0.013208121282148412 -0.14858702223380166 0.2541880957400964 rpy=-0.07907934249382903 -0.0520316044795478 0.2752784843541201
- added joint r_wrist_1_fixed_joint: type fixed, parent root_link, child r_wrist_1, origin xyz=0.045183921282148404 -0.16567102223380167 -0.030245004259903563 rpy=-0.07907934249382903 -0.0520316044795478 0.2752784843541201
- added joint torso_1_fixed_joint: type fixed, parent root_link, child torso_1, origin xyz=0 0 0.0605 rpy=0 -0 0
- added joint torso_2_fixed_joint: type fixed, parent root_link, child torso_2, origin xyz=0 0 0.133 rpy=0 -0 0
